File: pcb/splitboard.kicad_pcb (KiCad board)
At the start: 2 copper layers, 222.9 x 95.2 mm, 150 parts, among them IC1 ATMEGA32U4-MU, J1 Conn_02x05_Counter_Clockwise, J2 Conn_droite, J3 Conn_On_Off, Q1 Q_NPN_BCE, Q2 Q_NPN_BCE, SW1 SW_Push_LED, SW10 SW_Push_LED, SW101 SPST_TACT-KMR2, SW11 SW_Push_LED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

Commit message: pcb
Routing:
- net vcc1: track 175.1 -> 173.6 mm
